File: Hardware/telescope_driver.kicad_sch (KiCad schematic)
At the start: 63 parts, among them J1 GPIO, J2 Battery 12-14V, J3 Stepper_Motor_bipolar, J4 Stepper_Motor_bipolar, U1 TMC2209-LA, U2 TMC2209-LA, U3 LM2678S-12

Commit message: test
Parts:
- added R7: 1k, Resistor_SMD:R_1206_3216Metric_Pad1.30x1.75mm_HandSolder, symbol Device:R
Changed lines of the file:
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@@
+	)
+	(symbol
+		(lib_id "Device:R")
+		(at 60.96 196.85 0)
+		(unit 1)
+		(exclude_from_sim no)
+		(in_bom yes)
+		(on_board yes)
+		(dnp no)
+		(fields_autoplaced yes)
+		(property "Reference" "R7"
+			(at 63.5 195.5799 0)
+			(effects
+				(font
+					(size 1.27 1.27)
+				)
+				(justify left)
+			)
+		)
+		(property "Value" "1k"
+			(at 63.5 198.1199 0)
+			(effects
+				(font
+					(size 1.27 1.27)
+				)
+				(justify left)
+			)
+		)
+		(property "Footprint" "Resistor_SMD:R_1206_3216Metric_Pad1.30x1.75mm_HandSolder"
+			(at 59.182 196.85 90)
+			(effects
+				(font
+					(size 1.27 1.27)
+				)
+				(hide yes)
+			)
+		)
+		(property "Datasheet" "~"
+			(at 60.96 196.85 0)
+			(effects
+				(font
+					(size 1.27 1.27)
+				)
+				(hide yes)
+			)
+		)
+		(property "Description" "Resistor"
+			(at 60.96 196.85 0)
+			(effects
+				(font
+					(size 1.27 1.27)
+				)
+				(hide yes)
+			)
+		)
+		(pin "1"
+		)
+		(pin "2"
+		)
+		(instances
+			(project "telescope_driver"
+				(path "/e63e39d7-6ac0-4ffd-8aa3-1841a4541b55"
+					(reference "R7")
+					(unit 1)
+				)
+			)
+		)
 	)
 	(symbol

Commit message: update
Parts:
- removed R7: 1k, Resistor_SMD:R_1206_3216Metric_Pad1.30x1.75mm_HandSolder, symbol Device:R
Other:
- note added: "Raspberry Pi 5"
- note removed: "Pi"
Changed lines of the file:
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@@
 		)
 	)
-	(text "Pi"
+	(text "Raspberry Pi 5\n"
 		(exclude_from_sim no)
-		(at 21.336 20.066 0)
+		(at 29.972 17.78 0)
 		(effects
 			(font
@@
 	(wire
 		(pts
-			(xy 198.12 130.81) (xy 208.28 130.81)
+			(xy 205.74 130.81) (xy 208.28 130.81)
 		)
 		(stroke
@@
 	(wire
 		(pts
-			(xy 198.12 133.35) (xy 208.28 133.35)
+			(xy 187.96 133.35) (xy 208.28 133.35)
 		)
 		(stroke
@@
 	(wire
 		(pts
-			(xy 198.12 135.89) (xy 208.28 135.89)
+			(xy 193.04 135.89) (xy 208.28 135.89)
 		)
 		(stroke
@@
 	)
 	(label "UART"
-		(at 198.12 135.89 180)
+		(at 193.04 135.89 180)
 		(effects
 			(font
@@
 	)
 	(label "GPIO21{slash}PCM.DOUT"
-		(at 198.12 130.81 180)
+		(at 205.74 130.81 180)
 		(effects
 			(font
@@
 	)
 	(label "GPIO26"
-		(at 198.12 133.35 0)
+		(at 187.96 133.35 0)
 		(effects
 			(font
@@
 					(unit 1)
 				)
-			)
-		)
-	)
-	(symbol
-		(lib_id "Device:R")
-		(at 60.96 196.85 0)
-		(unit 1)
-		(exclude_from_sim no)
-		(in_bom yes)
-		(on_board yes)
-		(dnp no)
-		(fields_autoplaced yes)
-		(property "Reference" "R7"
-			(at 63.5 195.5799 0)
-			(effects
-				(font
-					(size 1.27 1.27)
-				)
-				(justify left)
-			)
-		)
-		(property "Value" "1k"
-			(at 63.5 198.1199 0)
-			(effects
-				(font
-					(size 1.27 1.27)
-				)
-				(justify left)
-			)
-		)
-		(property "Footprint" "Resistor_SMD:R_1206_3216Metric_Pad1.30x1.75mm_HandSolder"
-			(at 59.182 196.85 90)
-			(effects
-				(font
-					(size 1.27 1.27)
-				)
-				(hide yes)
-			)
-		)
-		(property "Datasheet" "~"
-			(at 60.96 196.85 0)
-			(effects
-				(font
-					(size 1.27 1.27)
-				)
-				(hide yes)
-			)
-		)
-		(property "Description" "Resistor"
-			(at 60.96 196.85 0)
-			(effects
-				(font
-					(size 1.27 1.27)
-				)
-				(hide yes)
-			)
-		)
-		(pin "1"
-		)
-		(pin "2"
-		)
-		(instances
-			(project "telescope_driver"
-				(path "/e63e39d7-6ac0-4ffd-8aa3-1841a4541b55"
-					(reference "R7")
-					(unit 1)
-				)

Commit message: some changes
Parts:
- added C31: 0.01 uF, Capacitor_SMD:C_0402_1005Metric_Pad0.74x0.62mm_HandSolder, symbol Device:C
- added R7, R8: 130, Resistor_SMD:R_1206_3216Metric_Pad1.30x1.75mm_HandSolder, symbol Device:R
Connections:
- net +5V: now also C31.1
- net GND: now also C31.2, R7.1, R8.1
- net at D2.1 (K), R4.2: no longer D4.1 (K)
- net at D1.1 (K), R5.2: no longer D6.1 (K)
- new net: D4.1 (K), R8.2
- new net: D6.1 (K), R7.2
Other:
- moved on the sheet: C12, C26, C27, C28, C29, C30, D11, D16, D5, F2, J2, L1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
