File: Hardware/telescope_driver.kicad_sch (KiCad schematic)
At the start: 66 parts, among them J1 GPIO, J2 Battery 12-14V, J3 Stepper_Motor_bipolar, J4 Stepper_Motor_bipolar, U1 TMC2209-LA, U2 TMC2209-LA, U3 LM2678S-12

Commit message: components ordered and some minor changes
Parts:
- R1: value 130 -> 0
- R3, R4, R5, R7, R8: value 130 -> 600
