File: Hardware/telescope_driver.kicad_pcb (KiCad board)
At the start: 2 copper layers, 67 x 56 mm, 66 parts, among them J1 GPIO, J2 Battery 12-14V, J3 Stepper_Motor_bipolar, J4 Stepper_Motor_bipolar, U1 TMC2209-LA, U2 TMC2209-LA, U3 LM2678S-12

Commit message: some changes
Parts:
- added C31: 0.01 uF, Capacitor_SMD:C_0402_1005Metric_Pad0.74x0.62mm_HandSolder, F.Cu at (137.8, 78.2)
- added R7: 130, Resistor_SMD:R_1206_3216Metric_Pad1.30x1.75mm_HandSolder, F.Cu at (162.6, 62.4)
- added R8: 130, Resistor_SMD:R_1206_3216Metric_Pad1.30x1.75mm_HandSolder, F.Cu at (137.1, 60.0)
- moved R5 9.66 mm to (161.1, 53.3), turned to 180 degrees
Connections:
- D4 pad 1: Net-(D2-K) -> Net-(D4-K)
- D6 pad 1: Net-(D1-K) -> Net-(D6-K)
Routing:
- net Net-(D6-K): track 0.00 -> 4.48 mm
- net Net-(D1-K): track 7.10 -> 2.96 mm
- net GND: track 151.6 -> 155.6 mm
- net Net-(D2-K): track 6.93 -> 4.48 mm
- net Net-(D4-K): track 0.00 -> 1.82 mm
- net +5V: track 65.2 -> 66.8 mm

Commit message: components ordered and some minor changes
Routing:
- net GND: vias 3 -> 19
Other:
- outline, holes or cut-outs redrawn
Changed lines of the file:
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@@
 		(grid_origin 100 100)
 		(pcbplotparams
-			(layerselection 0x00000000_00000000_00000000_000000a5)
+			(layerselection 0x00000000_00000000_55555555_5755f5ff)
 			(plot_on_all_layers_selection 0x00000000_00000000_00000000_00000000)
 			(disableapertmacros no)
@@
 			(outputformat 1)
 			(mirror no)
-			(drillshape 1)
+			(drillshape 0)
 			(scaleselection 1)
-			(outputdirectory "")
+			(outputdirectory "./")
 		)
 	)
@@
 		(at 143.7 61.05)
 		(property "Reference" "C7"
-			(at -4.55 -1.74 0)
+			(at -4.55 -1.65 0)
 			(layer "F.SilkS")
 			(effects
@@
 		)
 		(property "Value" "130"
-			(at 0 1.83 0)
+			(at -2.4876 1.864 0)
 			(layer "F.Fab")
 			(effects
@@
 		(layer "Edge.Cuts")
 	)
+	(gr_arc
+		(start 101 100)
+		(mid 98.87868 99.12132)
+		(end 98 97)
+		(stroke
+			(width 0.16)
+			(type default)
+		)
+		(layer "Edge.Cuts")
+	)
 	(gr_line
 		(start 103 44)
-		(end 98 44)
+		(end 101 44)
 		(stroke
 			(width 0.16)
@@
 		(layer "Edge.Cuts")
 	)
+	(gr_arc
+		(start 98 47)
+		(mid 98.87868 44.87868)
+		(end 101 44)
+		(stroke
+			(width 0.16)
+			(type default)
+		)
+		(layer "Edge.Cuts")
+	)
 	(gr_line
 		(start 147 81)
@@
 	(gr_line
 		(start 103 100)
-		(end 98 100)
+		(end 101 100)
 		(stroke
 			(width 0.16)
@@
 	)
 	(gr_line
-		(start 98 100)
-		(end 98 44)
+		(start 98 97)
+		(end 98 47)
 		(stroke
 			(width 0.16)
@@
 	)
 	(segment
+		(start 114.15 66.4)
+		(end 114.15 70.2)
+		(width 2)
+		(layer "F.Cu")
+		(net 1)
+	)
+	(segment
 		(start 125.55 59.8)
 		(end 126.55 58.8)
@@
 	(segment
 		(start 114.15 61.696653)
-		(end 114.15 79.812684)
+		(end 114.15 66.4)
 		(width 2)
 		(layer "F.Cu")
@@
 	)
 	(segment
+		(start 114.15 70.2)
+		(end 114.15 79.812684)
+		(width 2)
+		(layer "F.Cu")
+		(net 1)
+	)
+	(segment
 		(start 102.1 46.8)
 		(end 99.585 49.315)
@@
 	)
 	(via
+		(at 118.6 73.2)
+		(size 0.75)
+		(drill 0.2)
+		(layers "F.Cu" "B.Cu")
+		(free yes)
+		(net 1)
+	)
+	(via
+		(at 159.6 90.8)
+		(size 0.75)
+		(drill 0.2)
+		(layers "F.Cu" "B.Cu")
+		(free yes)
+		(net 1)
+	)
+	(via
+		(at 131.4 68.4)
+		(size 0.75)
+		(drill 0.2)
+		(layers "F.Cu" "B.Cu")
+		(free yes)
+		(net 1)
+	)
+	(via
+		(at 152 96.4)
+		(size 0.75)
+		(drill 0.2)
+		(layers "F.Cu" "B.Cu")
+		(free yes)
+		(net 1)
+	)
+	(via
 		(at 144.75 65.05)
 		(size 0.9)
@@
 	)
 	(via
+		(at 114.15 70.2)
+		(size 0.75)
+		(drill 0.2)
+		(layers "F.Cu" "B.Cu")
+		(net 1)
+	)
+	(via
+		(at 162.6 66.8)
+		(size 0.75)
+		(drill 0.2)
+		(layers "F.Cu" "B.Cu")
+		(free yes)
+		(net 1)
+	)
+	(via
+		(at 152 90.8)
+		(size 0.75)
+		(drill 0.2)
+		(layers "F.Cu" "B.Cu")
+		(free yes)
+		(net 1)
+	)
+	(via
+		(at 111.2 83.8)
+		(size 0.75)
+		(drill 0.2)
+		(layers "F.Cu" "B.Cu")
+		(free yes)
+		(net 1)
+	)
+	(via
+		(at 114.15 66.4)
+		(size 0.75)
+		(drill 0.2)
+		(layers "F.Cu" "B.Cu")
+		(net 1)
+	)
+	(via
+		(at 127.6 76.2)
+		(size 0.75)
+		(drill 0.2)
+		(layers "F.Cu" "B.Cu")
+		(free yes)
+		(net 1)
+	)
+	(via
+		(at 104.2 48.4)
+		(size 0.75)
+		(drill 0.2)
+		(layers "F.Cu" "B.Cu")
+		(free yes)
+		(net 1)
+	)
+	(via
+		(at 138 52.6)
+		(size 0.75)
+		(drill 0.2)
+		(layers "F.Cu" "B.Cu")
+		(free yes)
+		(net 1)
+	)
+	(via
+		(at 125 68.4)
+		(size 0.75)
+		(drill 0.2)
+		(layers "F.Cu" "B.Cu")
+		(free yes)
+		(net 1)
+	)
+	(via
+		(at 149.4 70.4)
+		(size 0.75)
+		(drill 0.2)
+		(layers "F.Cu" "B.Cu")
+		(free yes)
+		(net 1)
+	)
+	(via
+		(at 143.4 78.8)
+		(size 0.75)
+		(drill 0.2)
+		(layers "F.Cu" "B.Cu")
+		(free yes)
+		(net 1)
+	)
+	(via
 		(at 138.7 58.45)
 		(size 0.9)
@@
 		(net 1)
 	)
+	(via
+		(at 111.8 58.8)
+		(size 0.75)
+		(drill 0.2)
+		(layers "F.Cu" "B.Cu")
+		(free yes)
+		(net 1)
+	)
 	(segment
 		(start 143.35 63.1)
@@
 		(width 0.2)
 		(layer "F.Cu")
-		(net 59)
-	)
-	(segment
-		(start 128.75 48.83)
-		(end 128.69 48.77)
-		(width 0.2)
-		(layer "F.Cu")
